Commit message: hand-eye-calibration, eye-to-hand calibration code added

File: src/doosan-robot2/dsr_moveit_config_m1013_hande/config/m1013_hande.urdf.xacro (robot description, xacro)
@@ -2,8 +2,9 @@
 <robot xmlns:xacro="http://www.ros.org/wiki/xacro" name="m1013_hande">
     <xacro:arg name="use_gazebo" default="false"/>
-    <xacro:arg name="use_isaac"  default="true"/>
-    <xacro:arg name="use_real"   default="false"/>
+    <xacro:arg name="use_isaac"  default="false"/>
+    <xacro:arg name="use_real"   default="true"/>
+    <xacro:arg name="use_rviz"   default="false"/>
     <xacro:arg name="name" default="dsr01"/>
-    <xacro:arg name="host" default="192.168.56.1"/>
+    <xacro:arg name="host" default="192.168.137.100"/>
     <xacro:arg name="port" default="12345"/>
     <xacro:arg name="update_rate" default="100"/>
@@ -11,5 +12,6 @@
     <xacro:arg name="gripper_name" default="robotiq_hande"/>
     <xacro:arg name="gripper_prefix" default=""/>
-    <xacro:arg name="gripper_tty_port" default="/dev/ttyUSB0"/> <xacro:arg name="gripper_baudrate" default="115200"/>
+    <xacro:arg name="gripper_tty_port" default="/dev/ttyUSB0"/>
+    <xacro:arg name="gripper_baudrate" default="115200"/>
     <xacro:arg name="gripper_slave_id" default="9"/>
     <xacro:arg name="use_fake_gripper" default="false"/>
@@ -18,4 +20,5 @@
     <xacro:property name="use_isaac"   value="$(arg use_isaac)"/>
     <xacro:property name="use_real"    value="$(arg use_real)"/>
+    <xacro:property name="use_rviz"    value="$(arg use_rviz)"/>
     <xacro:property name="initial_positions_file" value="$(arg initial_positions_file)"/>
     <xacro:include filename="$(find dsr_description2)/xacro/m1013_hande.urdf.xacro" />
@@ -65,8 +68,64 @@
             frequency_hz="10.0"
             create_socat_tty="false"
-            socat_ip_address="192.168.1.1"
-            socat_port="33333"
+            socat_ip_address="192.168.137.100"
+            socat_port="54321"
             use_fake_hardware="false"
         />
     </xacro:if>
+    <xacro:if value="${use_rviz}">
+        <ros2_control name="RVizFakeSystem" type="system">
+            <hardware>
+                <plugin>mock_components/GenericSystem</plugin>
+            </hardware>
+            <joint name="joint_1">
+                <command_interface name="position"/>
+                <state_interface name="position">
+                    <param name="initial_value">0.0</param>
+                </state_interface>
+                <state_interface name="velocity"/>
+            </joint>
+            <joint name="joint_2">
+                <command_interface name="position"/>
+                <state_interface name="position">
+                    <param name="initial_value">0.0</param>
+                </state_interface>
+                <state_interface name="velocity"/>
+            </joint>
+            <joint name="joint_3">
+                <command_interface name="position"/>
+                <state_interface name="position">
+                    <param name="initial_value">1.57</param>
+                </state_interface>
+                <state_interface name="velocity"/>
+            </joint>
+            <joint name="joint_4">
+                <command_interface name="position"/>
+                <state_interface name="position">
+                    <param name="initial_value">0.0</param>
+                </state_interface>
+                <state_interface name="velocity"/>
+            </joint>
+            <joint name="joint_5">
+                <command_interface name="position"/>
+                <state_interface name="position">
+                    <param name="initial_value">1.57</param>
+                </state_interface>
+                <state_interface name="velocity"/>
+            </joint>
+            <joint name="joint_6">
+                <command_interface name="position"/>
+                <state_interface name="position">
+                    <param name="initial_value">0.0</param>
+                </state_interface>
+                <state_interface name="velocity"/>
+            </joint>
+            <joint name="robotiq_hande_left_finger_joint">
+                <command_interface name="position"/>
+                <state_interface name="position">
+                    <param name="initial_value">0.0</param>
+                </state_interface>
+                <state_interface name="velocity"/>
+            </joint>
+        </ros2_control>
+    </xacro:if>
 </robot>

File: src/robotiq_hande_description/urdf/robotiq_hande_gripper.urdf.xacro (robot description, xacro)
@@ -4,5 +4,5 @@
   <xacro:arg name="grip_pos_min" default="0"/>
   <xacro:arg name="grip_pos_max" default="0.025"/>
-  <xacro:arg name="tty_port" default="/tmp/ttyUR"/>
+  <xacro:arg name="tty_port" default="/dev/ttyUSB0"/>
   <xacro:arg name="baudrate" default="115200"/>
   <xacro:arg name="parity" default="N"/>

File: src/robotiq_hande_description/urdf/robotiq_hande_gripper.xacro (robot description, xacro)
@@ -26,5 +26,5 @@
             coupler_mass:=0.119
             xyz:='0 0 0'
-            rpy:='0 0 0'"
+            rpy:='0 0 1.57'"
   >
     <!-- ros2_control parameters  -->
